File: Hardware/source/KiCad/Archive/v00/PeterThePowerMeter.kicad_pcb (KiCad board)
At the start: 2 copper layers, 125.5 x 79 mm, 79 parts, among them J1 Screw_Terminal_01x02, J10 Conn_01x03_Pin, J11 Conn_01x03_Pin, J14 Conn_01x02_Pin, J15 Conn_01x02_Pin, J2 USB3076-30-A, J20 Conn_01x05_Pin, J21 Conn_01x05_Pin, J22 Conn_01x04_Male, J23 Conn_01x04_Male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

Commit message: Released 01 version
Parts:
- R21: value 220 -> 220R
- R24: value 1K -> 120
- R4: value 330 -> 330R
- moved R33 0.70 mm to (107.0, 101.8)
- moved TR1 0.70 mm to (103.5, 118.1)
- moved R30 0.50 mm to (113.8, 116.6)
- moved R28 0.32 mm to (115.9, 126.2)
- moved R29 0.10 mm to (115.9, 121.2)
Routing:
- net Net-(J3-Pin_2): track 11.0 -> 12.1 mm, vias 0 -> 1
- net Net-(R29-Pad1): track 3.82 -> 3.32 mm
Other:
- outline, holes or cut-outs redrawn
- rule pad_to_mask_clearance: 0.05 -> 0
- board text added: "04/2026"
- board text added: "250V 250mA T"
- board text added: "Base 15x79"
- board text added: "Right Side"
- board text added: "Sch.14 R.00"
- board text added: "Sch.14 R.00 04/2026"
- board text added: "TOP 15x38mm"
- board text removed: "250VAC 250mA T"
- board text removed: "LD1"
- board text removed: "SW1"
- board text removed: "SW2"
- board text removed: "Sch.14 R.01 06/2026"
