File: Hardware/source/KiCad/Archive/v00/PeterThePowerMeter.kicad_sch (KiCad schematic)
At the start: 79 parts, among them J1 Screw_Terminal_01x02, J10 Conn_01x03_Pin, J11 Conn_01x03_Pin, J14 Conn_01x02_Pin, J15 Conn_01x02_Pin, J2 USB3076-30-A, J20 Conn_01x05_Pin, J21 Conn_01x05_Pin, J22 Conn_01x04_Male, J23 Conn_01x04_Male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

Commit message: Released 01 version
Parts:
- BZ1: LCSC C49246960 -> (none)
- C1: LCSC C1580807 -> (none)
- C10, C6: LCSC C318754 -> (none)
- C11, C14, C2, C3, C5, C8, C9: LCSC C2167356 -> (none)
- C12, C13, C15: LCSC C89632 -> (none)
- C4: LCSC C1589590 -> (none)
- C7: LCSC C89632 -> (none); Note (none) -> CAP CER MLCC 10uF 50V X7R 1206
- D1, D2: LCSC C110921 -> (none)
- D3: LCSC C3018540 -> (none)
- F1: LCSC C3163460 -> (none)
- FB1: LCSC C840591 -> (none)
- J1, J3: LCSC C90074 -> (none)
- J2: LCSC C6007475 -> (none)
- J5: LCSC C2939183 -> (none)
- LD1: LCSC C133134 -> (none)
- Q1: LCSC C5184433 -> (none)
- R1, R2: LCSC C844876 -> (none)
- R10, R11, R12, R13, R14, R15, R18, R19, R20, R3, R31, R32, R6, R9: LCSC C132649 -> (none)
- R16, R17: LCSC C137394 -> (none)
- R21: value 220 -> 220R; LCSC C137353 -> (none)
- R22: LCSC C844863 -> (none)
- R23, R33: LCSC C131398 -> (none)
- R24: value 1K -> 120; LCSC C131398 -> (none)
- R28, R29, R30: LCSC C870906 -> (none)
- R4: value 330 -> 330R; LCSC C114944 -> (none)
- R5: LCSC C137392 -> (none)
- R7: LCSC C7233588 -> (none)
- R8: LCSC C2154230 -> (none)
- SW1: LCSC C470426 -> (none)
- SW2: LCSC C470426 -> (none); Note (none) -> 2 Alternative codes present in LCSC.com SKRPANE010 and C492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
- TH1: LCSC C75464 -> (none)
- TR1: LCSC C125191 -> (none)
- U1: LCSC C86781 -> (none)
- U2: LCSC C82891 -> (none)
- U3: LCSC C84681 -> (none)
- U4: LCSC C3194552 -> (none)
- U5: LCSC C37593 -> (none)
- U6: LCSC C7605 -> (none)
